Commit message: Comment

File: description/robot_core.xacro (robot description, xacro)
@@ -35,5 +35,5 @@
     </link>
     <!-- BASE_FOOTPRINT LINK -->
-    <joint name="base_footprint_joint" type="fixed">
+    <!-- <joint name="base_footprint_joint" type="fixed">
         <parent link="base_link"/>
         <child link="base_footprint"/>
@@ -41,5 +41,5 @@
     </joint>
     <link name="base_footprint">
-    </link>
+    </link> -->
     <!-- CHASSIS LINK -->
     <joint name="chassis_joint" type="fixed">

Commit message: Update caster_wheel_offset_z

File: description/robot_core.xacro (robot description, xacro)
@@ -11,9 +11,9 @@
     <xacro:property name="wheel_offset_x" value="0.315"/>
     <xacro:property name="wheel_offset_y" value="0.24"/>
-    <xacro:property name="wheel_offset_z" value="-0.03"/>
+    <xacro:property name="wheel_offset_z" value="0.03"/>
     <xacro:property name="caster_wheel_radius" value="0.035"/>
     <xacro:property name="caster_wheel_mass" value="0.200"/>
     <xacro:property name="caster_wheel_offset_x" value="0.71"/>
-    <xacro:property name="caster_wheel_offset_z" value="-0.035"/>
+    <xacro:property name="caster_wheel_offset_z" value="${wheel_offset_z - wheel_radius + caster_wheel_radius}"/>
     <material name="white">
         <color rgba="1 1 1 1" />

Commit message: Update robot_core.xacro

File: description/robot_core.xacro (robot description, xacro)
@@ -11,9 +11,9 @@
     <xacro:property name="wheel_offset_x" value="0.315"/>
     <xacro:property name="wheel_offset_y" value="0.24"/>
-    <xacro:property name="wheel_offset_z" value="0.03"/>
+    <xacro:property name="wheel_offset_z" value="-0.03"/>
     <xacro:property name="caster_wheel_radius" value="0.035"/>
     <xacro:property name="caster_wheel_mass" value="0.200"/>
     <xacro:property name="caster_wheel_offset_x" value="0.71"/>
-    <xacro:property name="caster_wheel_offset_z" value="${wheel_offset_z - wheel_radius + caster_wheel_radius}"/>
+    <xacro:property name="caster_wheel_offset_z" value="-0.035"/>
     <material name="white">
         <color rgba="1 1 1 1" />
@@ -35,5 +35,5 @@
     </link>
     <!-- BASE_FOOTPRINT LINK -->
-    <!-- <joint name="base_footprint_joint" type="fixed">
+    <joint name="base_footprint_joint" type="fixed">
         <parent link="base_link"/>
         <child link="base_footprint"/>
@@ -41,5 +41,5 @@
     </joint>
     <link name="base_footprint">
-    </link> -->
+    </link>
     <!-- CHASSIS LINK -->
     <joint name="chassis_joint" type="fixed">
